File: VESC_UI.sch (KiCad schematic (older format))
At the start: 92 parts, among them J1 Hall_SS443A, J2 Hall_SS443A, J3 Connector_Conn_01x04_Male, J4 Conn_01x05_Male, J5 Conn_01x07_Male, J6 Conn_01x04_Male, J7 USB_B_Micro, K1 K_0051, Q1 Q_0010-DVB_Q, Q2 Q_0010-DVB_Q, Q3 Q_0010-DVB_Q, Q4 Q_0010-DVB_Q, Q5 Q_0010-DVB_Q, Q6 Q_0010-DVB_Q, SW1 SW_Push, SW2 SW_Push, SW3 SW_Push, SW4 SW_Push, SW5 SW_Push, U1 U_0076, U2 STM32F401CEUx, Y1 8MHz

Commit message: Modify crystal type
Parts:
- removed R30: R_Small, symbol Device:R_Small
- removed Y1: 8MHz, symbol Device:Resonator_Small
- added C29, C30: C_Small, symbol Device:C_Small
- added Y1: Crystal_GND24_Small, symbol Device:Crystal_GND24_Small
- C24: Field6 16V -> 50V
Connections:
- wire segments 237 -> 243
Changed lines of the file:
@@
 Connection ~ 8125 1025
-$Comp
-L Device:Resonator_Small Y1
-U 1 1 5F5D9439
-P 6450 1975
-F 0 "Y1" V 6300 1975 50  0000 C CNN
-F 1 "8MHz" V 6425 2175 50  0000 C CNN
-F 2 "" H 6425 1975 50  0001 C CNN
-F 3 "~" H 6425 1975 50  0001 C CNN
-	1    6450 1975
-	0    1    1    0
-$EndComp
 $Comp
 L power:GND #PWR0123
 U 1 1 5F5E2B52
-P 6200 1975
-F 0 "#PWR0123" H 6200 1725 50  0001 C CNN
-F 1 "GND" H 6205 1802 50  0000 C CNN
-F 2 "" H 6200 1975 50  0001 C CNN
-F 3 "" H 6200 1975 50  0001 C CNN
-	1    6200 1975
-	1    0    0    -1
-$EndComp
-Wire Wire Line
-	6250 1975 6200 1975
-$Comp
-L Device:R_Small R30
-U 1 1 5F5E7FBC
-P 6650 2075
-F 0 "R30" V 6454 2075 50  0000 C CNN
-F 1 "R_Small" V 6725 2075 50  0000 C CNN
-F 2 "" H 6650 2075 50  0001 C CNN
-F 3 "~" H 6650 2075 50  0001 C CNN
-	1    6650 2075
-	0    1    1    0
+P 6550 2000
+F 0 "#PWR0123" H 6550 1750 39  0001 C CNN
+F 1 "GND" H 6550 1875 39  0000 C CNN
+F 2 "" H 6550 2000 39  0001 C CNN
+F 3 "" H 6550 2000 39  0001 C CNN
+	1    6550 2000
+	1    0    0    -1
 $EndComp
 NoConn ~ 7525 2225
@@
 $EndComp
 Wire Wire Line
-	7525 2025 6750 2025
-Wire Wire Line
-	6750 2025 6750 2075
-Wire Wire Line
-	7525 1925 6750 1925
-Wire Wire Line
-	6750 1925 6750 1875
-Wire Wire Line
-	6750 1875 6550 1875
+	7100 1925 7100 1875
 $Comp
 L power:+3.3V #PWR0144
@@
 P 9100 1100
 F 0 "#PWR0149" H 9100 850 50  0001 C CNN
-F 1 "GND" V 9105 972 30  0000 R CNN
+F 1 "GND" H 9150 975 30  0000 R CNN
 F 2 "" H 9100 1100 50  0001 C CNN
 F 3 "" H 9100 1100 50  0001 C CNN
@@
 F 4 "CER" H 6436 1255 0   0000 R CNN "Field4"
 F 5 "100nF" H 6550 1175 39  0000 R CNN "Field5"
-F 6 "16V" H 6550 1225 39  0000 R CNN "Field6"
+F 6 "50V" H 6550 1225 39  0000 R CNN "Field6"
 F 7 "X5R" H 6650 1150 60  0001 L CNN "Field7"
 F 8 "10%" H 6650 1075 60  0001 L CNN "Field8"
@@
 Wire Wire Line
 	6550 1450 6550 1400
+$Comp
+L Device:Crystal_GND24_Small Y1
+U 1 1 5F7C9C16
+P 6825 2000
+F 0 "Y1" V 6725 2025 39  0000 L CNN
+F 1 "Crystal_GND24_Small" V 6862 2144 39  0001 L CNN
+F 2 "" H 6825 2000 39  0001 C CNN
+F 3 "http://www.farnell.com/datasheets/2581422.pdf?_ga=2.29888511.1106248822.1601817720-706293543.1593275528&_gac=1.90918504.1601920666.CjwKCAjwiOv7BRBREiwAXHbv3Nre1ZRkFzw4o4_G1jayqOyIr5XBMbrn0P0vXxc_gtBymGv78yQuRBoCZ7kQAvD_BwE" H 6825 2000 39  0001 C CNN
+F 4 "8Mhz" V 6900 2075 28  0000 C CNN "Field4"
+F 5 "10ppm" V 6950 2100 28  0000 C CNN "Field5"
+	1    6825 2000
+	0    1    1    0
+$EndComp
+$Comp
+L Device:C_Small C29
+U 1 1 5F7DB934
+P 6725 1875
+F 0 "C29" V 6625 1875 39  0000 C CNN
+F 1 "C_Small" V 6587 1875 39  0001 C CNN
+F 2 "" H 6725 1875 39  0001 C CNN
+F 3 "~" H 6725 1875 39  0001 C CNN
+F 4 "15pf" V 6675 1800 28  0000 C CNN "Field4"
+F 5 "100v" V 6675 1950 28  0000 C CNN "Field5"
+	1    6725 1875
+	0    1    1    0
+$EndComp
+$Comp
+L Device:C_Small C30
+U 1 1 5F7DEDB9
+P 6725 2125
+F 0 "C30" V 6825 2125 39  0000 C CNN
+F 1 "C_Small" V 6587 2125 39  0001 C CNN
+F 2 "" H 6725 2125 39  0001 C CNN
+F 3 "~" H 6725 2125 39  0001 C CNN
+F 4 "15pf" V 6775 2050 28  0000 C CNN "Field4"
+F 5 "100v" V 6775 2200 28  0000 C CNN "Field5"
+	1    6725 2125
+	0    1    1    0
+$EndComp
+$Comp
+L power:GND #PWR05
+U 1 1 5F8237D6
+P 6925 2000
+F 0 "#PWR05" H 6925 1750 39  0001 C CNN
+F 1 "GND" H 6925 1875 39  0000 C CNN
+F 2 "" H 6925 2000 39  0001 C CNN
+F 3 "" H 6925 2000 39  0001 C CNN
+	1    6925 2000
+	0    -1   -1   0
+$EndComp
+Wire Wire Line
+	6825 1875 6825 1900
+Wire Wire Line
+	6825 2125 6825 2100
+Wire Wire Line
+	6625 1875 6625 2000
+Wire Wire Line
+	6625 2000 6725 2000
+Connection ~ 6625 2000
+Wire Wire Line
+	6625 2000 6625 2125
+Wire Wire Line
+	6625 2000 6550 2000
+Wire Wire Line
+	7100 2125 6825 2125
+Wire Wire Line
+	7100 2025 7100 2125
+Connection ~ 6825 2125
+Wire Wire Line
+	6825 1875 7100 1875
+Connection ~ 6825 1875
+Wire Wire Line
+	7525 1925 7100 1925
+Wire Wire Line
+	7100 2025 7525 2025
 $EndSCHEMATC

Commit message: Add RTC and buzzers
Parts:
- removed C18, C19, C20, C21, C22: C_Small, symbol Device:C_Small
- removed C3, C6, C8, C9: C_0002, DVB_Capacitors_Ceramic:C_0402, symbol Device:C
- removed Q1, Q3, Q4, Q5, Q6: Q_0010-DVB_Q, DVB_SOT:SOT_23, symbol VESC_UI-rescue:Q_0010-DVB_Q
- removed R10, R13, R14, R17, R2, R21, R26, R3: R_0020, DVB_Resistors:R_0402, symbol Device:R
- removed R15, R19, R24, R27, R4, R9: R_Small, symbol Device:R_Small
- added C22: CP_Small, symbol Device:Battery_Cell
- added C23: C_0033, symbol Device:C_Small
- added D10: D_Schottky_Small_ALT, symbol Device:D_Schottky_Small_ALT
- added J8, J9: Conn_01x02_Male, symbol Connector:Conn_01x02_Male
- added JP1, JP2: Jumper_NC_Small, symbol Device:Jumper_NC_Small
- added Q2: Q_0010-DVB_Q, DVB_SOT:SOT_23, symbol VESC_UI-rescue:Q_0010-DVB_Q
- added R1, R19, R20, R4: R_0020, DVB_Resistors:R_0402, symbol Device:R
- R17: renamed from R28; Field4 100 -> 0
- R18: renamed from R29; Field4 100 -> 0
- R6: Field4 10k -> 30
- renumbered C15 to C10, C12 to C11, C23 to C12, C16 to C14, C24 to C15, C29 to C16, C30 to C17, C25 to C18, C26 to C19, C27 to C20, C28 to C21, C4 to C3, C5 to C4, C7 to C5, C17 to C6, C10 to C7, C11 to C8, C14 to C9, D6 to D3, D7 to D4, D8 to D5, D9 to D6, D3 to D7, D4 to D8, D5 to D9, J5 to J3, J3 to J4, J4 to J5, Q2 to Q1, R16 to R10, R18 to R11, R20 to R12, R22 to R13, R23 to R14, R25 to R15, R31 to R16, R7 to R2, R1 to R3, R8 to R7, R11 to R8, R12 to R9
Connections:
- net labels added: Accelerator, BUZZER, Brake
- wire segments 243 -> 210
- no-connect marks 18 -> 17
Other:
- note added: "Buzzers"
- note added: "HMI"
- note added: "Light LEDS"
- note added: "OLED Power"
- note removed: "50"
- note removed: "IHM"
- note removed: "Power"
- moved on the sheet: C10, C6, C9, D1, D2, D3, D4, D5, D6, J1, J2, J3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

Commit message: first finished version
Parts:
- removed C1: C_0003, DVB_Capacitors_Ceramic:C_0603, symbol VESC_UI-rescue:C_0003-DVB_C
- removed C11, C5: C_0056, DVB_Capacitors_Ceramic:C_0805, symbol Device:C
- removed C13, C2: C_0033, DVB_Capacitors_Ceramic:C_0603, symbol Device:C
- removed C14, C4: C_0036, DVB_Capacitors_Ceramic:C_0603, symbol Device:C
- removed C3: C_0041, DVB_Capacitors_Ceramic:C_1206, symbol Device:C
- removed C7: C_0013, DVB_Capacitors_Ceramic:C_0402, symbol VESC_UI-rescue:C_0013-DVB_C
- removed C8: C_0036, DVB_Capacitors_Ceramic:C_0603, symbol VESC_UI-rescue:C_0036-DVB_C
- removed D7, D8: D_0022, DVB_Diodes:D_SOD-523, symbol Diode:1N4148WT
- removed D9: D_0021, DVB_Diodes:D_SOD-123, symbol VESC_UI-rescue:D_0021-DVB_D
- removed J4: Connector_Conn_01x04_Male, symbol VESC_UI-cache:Connector_Conn_01x04_Male
- removed J7: USB_B_Micro, symbol Connector:USB_B_Micro
- removed K1: K_0051, DVB_Displays:OLED128x128-1P5, symbol VESC_UI-rescue:K_0051-DVB_K-DK3_GUI-PI-rescue
- removed L1: L_0011, DVB_Inductors:L_4018-Coilcraft, symbol Device:L
- removed R10: R_0107, DVB_Resistors:R_0402, symbol VESC_UI-rescue:R_0107-DVB_R
- removed R11: R_0108, DVB_Resistors:R_0402, symbol VESC_UI-rescue:R_0108-DVB_R
- removed R15: R_0019, DVB_Resistors:R_0402, symbol Device:R
- removed R8: R_0110, DVB_Resistors:R_0402, symbol Device:R
- removed U1: U_0076, Package_TO_SOT_SMD:SOT-23-5, symbol VESC_UI-rescue:U_0076-DVB_U
- added C24: C_0033, Capacitor_SMD:C_0603_1608Metric_Pad1.05x0.95mm_HandSolder, symbol Device:C_Small
- added J4: Conn_01x09_Female, Connector_PinHeader_1.27mm:PinHeader_1x09_P1.27mm_Vertical, symbol Connector:Conn_01x09_Female
- added R21, R22: R_Small, Resistor_SMD:R_0603_1608Metric_Pad1.05x0.95mm_HandSolder, symbol Device:R_Small
- added U3: M95M04-DR, Package_SO:SOIC-8_3.9x4.9mm_P1.27mm, symbol Memory_EEPROM:M95256-WMN6P
- C10, C12, C15, C16, C17, C19, C20, C21, C23, C6, C9: footprint (none) -> Capacitor_SMD:C_0603_1608Metric_Pad1.05x0.95mm_HandSolder
- C18: value 2.2u -> 4.7u; footprint (none) -> Capacitor_SMD:C_0603_1608Metric_Pad1.05x0.95mm_HandSolder
- C22: footprint (none) -> SamacSys_Parts:DSK3R3H334THL
- D1, D2, D3, D4, D5, D6: footprint (none) -> LED_THT:LED_D5.0mm_Clear
- D10: footprint (none) -> Diode_SMD:D_0603_1608Metric_Pad1.05x0.95mm_HandSolder
- J5: footprint (none) -> Connector_JST:JST_PH_B5B-PH-K_1x05_P2.00mm_Vertical
- J6: footprint (none) -> Connector_JST:JST_PH_B4B-PH-K_1x04_P2.00mm_Vertical
- J8, J9: footprint (none) -> Connector_JST:JST_PH_B2B-PH-K_1x02_P2.00mm_Vertical
- JP1, JP2: footprint (none) -> Jumper:SolderJumper-2_P1.3mm_Open_TrianglePad1.0x1.5mm
- L2: value L_Core_Iron_Small -> MMZ1608B121C; footprint (none) -> Inductor_SMD:L_0603_1608Metric_Pad1.05x0.95mm_HandSolder; Field4 1KOhm -> 120Ohm; Field6 10% -> 25%
- Q1, Q2: footprint DVB_SOT:SOT_23 -> Package_TO_SOT_SMD:SOT-23
- R1, R14, R19, R2, R20, R4, R6: footprint DVB_Resistors:R_0402 -> Resistor_SMD:R_0603_1608Metric_Pad1.05x0.95mm_HandSolder
- R12, R16, R17, R18, R3, R5, R7, R9: footprint (none) -> Resistor_SMD:R_0603_1608Metric_Pad1.05x0.95mm_HandSolder
- R13: footprint (none) -> Resistor_THT:R_Axial_DIN0204_L3.6mm_D1.6mm_P2.54mm_Vertical
- SW1, SW2, SW3, SW4: footprint (none) -> SamacSys_Parts:Vertical_push_button
- Y1: footprint (none) -> Crystal:Crystal_SMD_Abracon_ABM3B-4Pin_5.0x3.2mm
Connections:
- net labels added: EXT_FLASH_CS, SPI1_MISO, SPI1_MOSI, SPI1_SCK
- net labels removed: I2C1_SCL, I2C1_SDA, OLED_DIN, OLED_SCK, USB_D+, USB_D-
- wire segments 210 -> 160
- no-connect marks 17 -> 12
Other:
- note removed: "OLED Power"
- note removed: "OLED SCREEN"
