File: VESC_UI.sch (KiCad schematic (older format))
At the start: 57 parts, among them J1 Hall_SS441R, J2 Hall_SS441R, J3 Conn_01x07_Male, J4 Conn_02x05_Female, J5 Conn_01x05_Male, J6 Conn_01x04_Male, J8 Conn_01x02_Male, J9 Conn_01x02_Male, Q1 Mosfet IRLML2060TRPBF, Q2 Mosfet IRLML2060TRPBF, SW1 Vertical push button, SW2 Vertical push button, SW3 Vertical push button, SW4 Vertical push button, SW5 Push button, U2 STM32F401CEU6, U3 M95M04-DR

Commit message: fix(Mainboard): LEDs not working due to insufficient current
Parts:
- added R10, R11, R15: 62, Resistor_SMD:R_0603_1608Metric_Pad1.05x0.95mm_HandSolder, symbol Device:R_Small
- C2: symbol VESC_UI-rescue:C_0003-DVB_C -> Device:C
- J1, J2: value Hall_SS441R -> Hall_DRV5055-Q1
- R1, R4, R6: value 30 -> 62; symbol Device:R -> Device:R_Small
- R14, R2: symbol Device:R -> Device:R_Small
Connections:
- net +12V: no longer Q2.3 (D)
- net +5V: now also D2.2 (A), D4.2 (A), D6.2 (A)
- net GND: no longer J8.2 (Pin_2), J9.2 (Pin_2)
- net at Q1.3 (D), R1.2, R4.2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: now also R10.2, R11.2, R15.2
- net at D1.1 (K): now also R1.1; no longer D2.2 (A)
- net at D2.1 (K): now also R10.1; no longer R1.1
- net at D3.1 (K): now also R11.1; no longer D4.2 (A)
- net at D4.1 (K): now also R15.1; no longer R4.1
- net at D5.1 (K): now also R4.1; no longer D6.2 (A)
- new net: J8.2 (Pin_2), J9.2 (Pin_2), Q2.3 (D)
Other:
- moved on the sheet: C1, C12, C23, C6, D1, D2, D3, D4, D5, D6, J8, J9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
