File: VESC_UI.kicad_sch (KiCad schematic)
At the start: 86 parts, among them IC1 FAN5331SX, J1 Hall_DRV5055-Q1, J2 Hall_DRV5055-Q1, J3 Conn_01x07_Male, J5 Conn_01x05_Male, J6 Conn_01x04_Male, J8 Conn_01x02_Male, J9 Conn_01x02_Male, K1 K_0051-OBSOLETE, Q1 Q_0020, Q2 Q_0020, SW1 Vertical push button, SW2 Vertical push button, SW3 Vertical push button, SW4 Vertical push button, SW5 SW_0002, U2 STM32F401CEUx, U3 M95M04-DR

Commit message: Route complete
Parts:
- removed C7: C_0036, DVB_Capacitors_Ceramic:C_0603, symbol DVB_C:C_0036
- removed SW5: SW_0002, DVB_Buttons:KSS221G, symbol DVB_SW:SW_0002
- added C7: C_0003, DVB_Capacitors_Ceramic:C_0603, symbol DVB_C:C_0003
- added SW5: SW_0003, DVB_Buttons:PTS810, symbol DVB_SW:SW_0003
Connections:
- net GND: now also C7.2, SW5.3
- net NRST: now also SW5.2
- net at K1.3 (VCOMH): now also C7.1
Changed lines of the file:
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@@
   (title_block
     (title "VESC_UI")
-    (date "2021-07-21")
+    (date "2021-08-06")
     (rev "2.0.0")
   )
@@
     (pin "2")
   )
-  (symbol (lib_id "DVB_SW:SW_0002") (at 127 33.655 270) (unit 1)
-    (in_bom yes) (on_board yes)
-    (property "Reference" "SW5" (id 0) (at 129.794 37.465 0))
-    (property "Value" "SW_0002" (id 1) (at 121.92 33.655 0)
-      (effects (font (size 1.27 1.27)) hide)
-    )
-    (property "Footprint" "DVB_Buttons:KSS221G" (id 2) (at 116.84 33.655 0)
-      (effects (font (size 1.27 1.27)) hide)
-    )
-    (property "Datasheet" "https://www.mouser.fr/datasheet/2/60/kss-965434.pdf" (id 3) (at 119.38 33.655 0)
-      (effects (font (size 1.27 1.27)) hide)
-    )
-    (property "Field4" "KSS221GLFS" (id 4) (at 124.46 34.925 0))
-    (property "Field5" "PUSH BUTTON" (id 5) (at 114.3 33.655 0)
-      (effects (font (size 1.1176 1.1176)) hide)
-    )
-    (property "Field6" "SPST-NO" (id 6) (at 127 33.655 0)
-      (effects (font (size 0 0)) (justify left))
-    )
-    (property "Field7" "RA" (id 7) (at 111.76 33.655 0)
-      (effects (font (size 1.1176 1.1176)) hide)
-    )
-    (pin "1")
-    (pin "2")
-  )
   (symbol (lib_id "Connector:Conn_01x03_Female") (at 156.21 127 0) (unit 1)
     (in_bom yes) (on_board yes)
@@
     (pin "2")
   )
-  (symbol (lib_id "DVB_C:C_0036") (at 38.735 89.535 0) (mirror y) (unit 1)
+  (symbol (lib_id "DVB_C:C_0003") (at 38.735 89.535 0) (unit 1)
     (in_bom yes) (on_board yes)
-    (property "Reference" "C7" (id 0) (at 36.195 87.63 0)
+    (property "Reference" "C7" (id 0) (at 41.275 87.63 0)
       (effects (font (size 1.27 1.27)) (justify left))
     )
-    (property "Value" "C_0036" (id 1) (at 38.735 97.155 0)
+    (property "Value" "C_0003" (id 1) (at 38.735 97.155 0)
       (effects (font (size 1.27 1.27)) hide)
     )
@@
       (effects (font (size 0 0)) (justify left))
     )
-    (property "Field5" "4.7µF" (id 5) (at 36.195 89.535 0)
+    (property "Field5" "10µF" (id 5) (at 41.275 89.535 0)
       (effects (font (size 1.27 1.27)) (justify left))
     )
-    (property "Field6" "25V" (id 6) (at 36.195 91.44 0)
+    (property "Field6" "25V" (id 6) (at 41.275 91.44 0)
       (effects (font (size 1.27 1.27)) (justify left))
     )
-    (property "Field7" "X5R" (id 7) (at 36.195 93.345 0)
+    (property "Field7" "X5R" (id 7) (at 41.275 93.345 0)
       (effects (font (size 1.524 1.524)) (justify left) hide)
     )
-    (property "Field8" "10%" (id 8) (at 36.195 95.25 0)
+    (property "Field8" "10%" (id 8) (at 41.275 95.25 0)
       (effects (font (size 1.524 1.524)) (justify left) hide)
     )
@@
     (pin "7")
   )
+  (symbol (lib_id "DVB_SW:SW_0003") (at 132.08 33.655 270) (unit 1)
+    (in_bom yes) (on_board yes)
+    (property "Reference" "SW5" (id 0) (at 136.525 33.655 0))
+    (property "Value" "SW_0003" (id 1) (at 114.3 33.655 0)
+      (effects (font (size 1.27 1.27)) hide)
+    )
+    (property "Footprint" "DVB_Buttons:PTS810" (id 2) (at 116.84 33.655 0)
+      (effects (font (size 1.27 1.27)) hide)
+    )
+    (property "Datasheet" "https://www.ckswitches.com/media/1476/pts810.pdf" (id 3) (at 119.38 33.655 0)
+      (effects (font (size 1.27 1.27)) hide)
+    )
+    (property "Field1" "PTS810" (id 4) (at 124.46 33.655 0))
+    (property "Field2" "PUSH BUTTON" (id 5) (at 111.76 33.655 0)
+      (effects (font (size 1.27 1.27)) hide)
+    )
+    (property "Field3" "DPST-NO" (id 6) (at 109.22 33.655 0)
+      (effects (font (size 1.27 1.27)) hide)
+    )
+    (property "Field7" "TOP" (id 7) (at 106.68 33.655 0)
+      (effects (font (size 1.27 1.27)) hide)
+    )
+    (pin "1")
+    (pin "2")
+    (pin "3")
+    (pin "4")
+  )
   (symbol (lib_id "SamacSys_Parts:FAN5331SX") (at 57.15 33.655 0) (mirror y) (unit 1)
     (in_bom yes) (on_board yes)
@@
     (pin "9")
   )
-  (symbol (lib_name "MCU_ST_STM32F4:STM32F401CEUx_1") (lib_id "MCU_ST_STM32F4:STM32F401CEUx") (at 212.725 85.725 0) (unit 1)
+  (symbol (lib_id "MCU_ST_STM32F4:STM32F401CEUx") (at 212.725 85.725 0) (unit 1)
     (in_bom yes) (on_board yes)
     (property "Reference" "U2" (id 0) (at 222.885 46.355 0)
@@
       (reference "C6") (unit 1) (value "C_0002") (footprint "DVB_Capacitors_Ceramic:C_0402")
     )
-    (path "/93538aff-e433-4103-8ee0-f61ee1ef8c1d"
-      (reference "C7") (unit 1) (value "C_0036") (footprint "DVB_Capacitors_Ceramic:C_0603")
+    (path "/06bde163-f815-496e-9483-f2f8f10a9b5b"
+      (reference "C7") (unit 1) (value "C_0003") (footprint "DVB_Capacitors_Ceramic:C_0603")
     )
     (path "/7d3e3916-a429-4804-9b19-4cc80f965da4"
@@
       (reference "SW4") (unit 1) (value "Vertical push button") (footprint "SamacSys_Parts:Vertical_push_button")
     )
-    (path "/e5d0da17-848c-4a39-a6f4-a97ae118eff9"
-      (reference "SW5") (unit 1) (value "SW_0002") (footprint "DVB_Buttons:KSS221G")
+    (path "/2667c678-1acb-4ac1-86df-f5db22fc0242"
+      (reference "SW5") (unit 1) (value "SW_0003") (footprint "DVB_Buttons:PTS810")
     )
     (path "/6d0ff79b-0241-4693-a6ac-4fd600ca2613"

Commit message: v2.0.0 version
Parts:
- R1, R10, R11, R15, R4, R6: footprint DVB_Resistors:R_0402 -> DVB_Resistors:R_0603
- SW1, SW2, SW3, SW4: footprint SamacSys_Parts:Vertical_push_button -> DVB_Buttons:Vertical_push_button
Changed lines of the file:
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@@
       (effects (font (size 1.27 1.27)) hide)
     )
-    (property "Footprint" "DVB_Resistors:R_0402" (id 2) (at 19.05 149.225 0)
+    (property "Footprint" "DVB_Resistors:R_0603" (id 2) (at 19.05 149.225 0)
       (effects (font (size 1.27 1.27)) hide)
     )
@@
       (effects (font (size 1.27 1.27)) hide)
     )
-    (property "Footprint" "DVB_Resistors:R_0402" (id 2) (at 24.13 149.225 0)
+    (property "Footprint" "DVB_Resistors:R_0603" (id 2) (at 24.13 149.225 0)
       (effects (font (size 1.27 1.27)) hide)
     )
@@
       (effects (font (size 1.27 1.27)) hide)
     )
-    (property "Footprint" "DVB_Resistors:R_0402" (id 2) (at 29.21 149.225 0)
+    (property "Footprint" "DVB_Resistors:R_0603" (id 2) (at 29.21 149.225 0)
       (effects (font (size 1.27 1.27)) hide)
     )
@@
       (effects (font (size 1.27 1.27)) hide)
     )
-    (property "Footprint" "DVB_Resistors:R_0402" (id 2) (at 34.29 149.225 0)
+    (property "Footprint" "DVB_Resistors:R_0603" (id 2) (at 34.29 149.225 0)
       (effects (font (size 1.27 1.27)) hide)
     )
@@
       (effects (font (size 1.27 1.27)) hide)
     )
-    (property "Footprint" "DVB_Resistors:R_0402" (id 2) (at 39.37 149.225 0)
+    (property "Footprint" "DVB_Resistors:R_0603" (id 2) (at 39.37 149.225 0)
       (effects (font (size 1.27 1.27)) hide)
     )
@@
       (effects (font (size 1.27 1.27)) hide)
     )
-    (property "Footprint" "DVB_Resistors:R_0402" (id 2) (at 44.45 149.225 0)
+    (property "Footprint" "DVB_Resistors:R_0603" (id 2) (at 44.45 149.225 0)
       (effects (font (size 1.27 1.27)) hide)
     )
@@
       (effects (font (size 0.9906 0.9906)) (justify right) hide)
     )
-    (property "Footprint" "SamacSys_Parts:Vertical_push_button" (id 2) (at 106.045 139.7 0)
+    (property "Footprint" "DVB_Buttons:Vertical_push_button" (id 2) (at 106.045 139.7 0)
       (effects (font (size 0.9906 0.9906)) hide)
     )
@@
       (effects (font (size 0.9906 0.9906)) (justify right) hide)
     )
-    (property "Footprint" "SamacSys_Parts:Vertical_push_button" (id 2) (at 106.045 172.085 0)
+    (property "Footprint" "DVB_Buttons:Vertical_push_button" (id 2) (at 106.045 172.085 0)
       (effects (font (size 0.9906 0.9906)) hide)
     )
@@
       (effects (font (size 0.9906 0.9906)) (justify right) hide)
     )
-    (property "Footprint" "SamacSys_Parts:Vertical_push_button" (id 2) (at 122.555 139.7 0)
+    (property "Footprint" "DVB_Buttons:Vertical_push_button" (id 2) (at 122.555 139.7 0)
       (effects (font (size 0.9906 0.9906)) hide)
     )
@@
       (effects (font (size 0.9906 0.9906)) (justify right) hide)
     )
-    (property "Footprint" "SamacSys_Parts:Vertical_push_button" (id 2) (at 122.555 172.085 0)
+    (property "Footprint" "DVB_Buttons:Vertical_push_button" (id 2) (at 122.555 172.085 0)
       (effects (font (size 0.9906 0.9906)) hide)
     )
@@
     )
     (path "/274f8f4b-6844-4f32-8ecc-3b008e20dab4"
-      (reference "R1") (unit 1) (value "R_0110") (footprint "DVB_Resistors:R_0402")
+      (reference "R1") (unit 1) (value "R_0110") (footprint "DVB_Resistors:R_0603")
     )
     (path "/fc81d31a-d19a-45e9-b1d9-0dbd0d552d01"
@@
     )
     (path "/cc694b3e-764f-4afb-a606-e4bea4e60d84"
-      (reference "R4") (unit 1) (value "R_0110") (footprint "DVB_Resistors:R_0402")
+      (reference "R4") (unit 1) (value "R_0110") (footprint "DVB_Resistors:R_0603")
     )
     (path "/73172fa1-a555-4a52-a7e5-d156d096e84c"
@@
     )
     (path "/2a3fd3fe-ce9c-4f48-87f2-1e093761143a"
-      (reference "R6") (unit 1) (value "R_0110") (footprint "DVB_Resistors:R_0402")
+      (reference "R6") (unit 1) (value "R_0110") (footprint "DVB_Resistors:R_0603")
     )
     (path "/b30ecf8e-a8fc-4661-b6ea-8889d18687dc"
@@
     )
     (path "/210b967b-f808-421a-b093-846820131e84"
-      (reference "R10") (unit 1) (value "R_0110") (footprint "DVB_Resistors:R_0402")
+      (reference "R10") (unit 1) (value "R_0110") (footprint "DVB_Resistors:R_0603")
     )
     (path "/1e416a78-27a3-4ff1-925a-5ba0932f03a7"
-      (reference "R11") (unit 1) (value "R_0110") (footprint "DVB_Resistors:R_0402")
+      (reference "R11") (unit 1) (value "R_0110") (footprint "DVB_Resistors:R_0603")
     )
     (path "/fc3cd660-2089-4bf6-a20f-d1d131f3fc27"
@@
     )
     (path "/7146dc1d-217b-4ba2-a470-61e4a0cc9a7c"
-      (reference "R15") (unit 1) (value "R_0110") (footprint "DVB_Resistors:R_0402")
+      (reference "R15") (unit 1) (value "R_0110") (footprint "DVB_Resistors:R_0603")
     )
     (path "/c79941fd-6173-4b87-8e18-a7e29ac12dea"
@@
     )
     (path "/00000000-0000-0000-0000-00005f5cdcd2"
-      (reference "SW1") (unit 1) (value "Vertical push button") (footprint "SamacSys_Parts:Vertical_push_button")
+      (reference "SW1") (unit 1) (value "Vertical push button") (footprint "DVB_Buttons:Vertical_push_button")
     )
     (path "/4c24bb6c-4be8-4832-bb7d-19e358013a23"
-      (reference "SW2") (unit 1) (value "Vertical push button") (footprint "SamacSys_Parts:Vertical_push_button")
+      (reference "SW2") (unit 1) (value "Vertical push button") (footprint "DVB_Buttons:Vertical_push_button")
     )
     (path "/4f42f5bd-6f0a-4547-86cd-71576a3d2ad3"
-      (reference "SW3") (unit 1) (value "Vertical push button") (footprint "SamacSys_Parts:Vertical_push_button")
+      (reference "SW3") (unit 1) (value "Vertical push button") (footprint "DVB_Buttons:Vertical_push_button")
     )
     (path "/05aafbf7-38b1-46f3-8fef-03cf38751b32"
-      (reference "SW4") (unit 1) (value "Vertical push button") (footprint "SamacSys_Parts:Vertical_push_button")
+      (reference "SW4") (unit 1) (value "Vertical push button") (footprint "DVB_Buttons:Vertical_push_button")
     )
     (path "/2667c678-1acb-4ac1-86df-f5db22fc0242"
